Commit message: Replace placeholder paddle robot with first quadruped Gizmo model
Iteration 1 simulation body: a body_link with head, four legs (hip +
knee per leg) and two arms, all driven by a single
joint_trajectory_controller exposing 10 revolute joints. Geometry is
boxes/cylinders/spheres so the controller pipeline can be validated
before real meshes arrive.

- new leg macro and materials xacro
- gizmo_joint_trajectory_controller replaces paddle_position_controller
- launch file spawns the new controller
- gizmo_gait_node.py scaffold publishes stand_pose / wave trajectories

File: src/gizmo_description/urdf/gizmo.urdf.xacro (robot description, xacro)
@@ -1,55 +1,112 @@
 <?xml version="1.0"?>
 <robot name="gizmo" xmlns:xacro="http://www.ros.org/wiki/xacro">
-  <!-- Placeholder skeleton: a base + one revolute joint + a paddle.
-       Replace with the real Gizmo geometry as it firms up. -->
-  <!-- controllers_yaml is resolved by the launch file via xacro mappings -->
+  <!--
+    Iteration 1 Gizmo: a simple quadruped with two arms.
+    Joints exposed to ros2_control:
+      front_left_hip_joint, front_left_knee_joint
+      front_right_hip_joint, front_right_knee_joint
+      rear_left_hip_joint,  rear_left_knee_joint
+      rear_right_hip_joint, rear_right_knee_joint
+      left_arm_joint, right_arm_joint
+    Geometry is deliberately box/cylinder/sphere only - this is here
+    to validate URDF, controllers and gait scaffolding, not to look
+    pretty. Real meshes come in a later iteration.
+  -->
   <xacro:arg name="controllers_yaml" default="/tmp/gizmo_controllers.yaml"/>
-  <xacro:property name="base_size" value="0.6 0.6 0.2"/>
-  <link name="base_link">
+  <xacro:include filename="$(find gizmo_description)/urdf/materials.xacro"/>
+  <xacro:include filename="$(find gizmo_description)/urdf/leg_macro.xacro"/>
+  <!-- Body geometry. -->
+  <xacro:property name="body_x" value="0.20"/>
+  <xacro:property name="body_y" value="0.15"/>
+  <xacro:property name="body_z" value="0.10"/>
+  <!-- Leg attachment offsets (relative to body_link). -->
+  <xacro:property name="hip_x" value="0.085"/>
+  <xacro:property name="hip_y" value="0.080"/>
+  <xacro:property name="hip_z" value="-0.04"/>
+  <!-- Root link: empty so Gazebo treats it as a free-floating base. -->
+  <link name="base_link"/>
+  <link name="body_link">
     <inertial>
-      <mass value="5.0"/>
+      <mass value="1.2"/>
       <origin xyz="0 0 0"/>
-      <inertia ixx="0.2" iyy="0.2" izz="0.2" ixy="0" ixz="0" iyz="0"/>
+      <inertia ixx="0.004" iyy="0.006" izz="0.008" ixy="0" ixz="0" iyz="0"/>
     </inertial>
     <visual>
-      <geometry><box size="${base_size}"/></geometry>
-      <material name="grey"><color rgba="0.5 0.5 0.5 1"/></material>
+      <geometry><box size="${body_x} ${body_y} ${body_z}"/></geometry>
+      <material name="gizmo_body"/>
     </visual>
     <collision>
-      <geometry><box size="${base_size}"/></geometry>
+      <geometry><box size="${body_x} ${body_y} ${body_z}"/></geometry>
     </collision>
   </link>
-  <link name="paddle_link">
+  <joint name="base_to_body" type="fixed">
+    <parent link="base_link"/>
+    <child link="body_link"/>
+    <origin xyz="0 0 0" rpy="0 0 0"/>
+  </joint>
+  <!-- Head: fixed for now, gets a joint in a later iteration. -->
+  <link name="head_link">
     <inertial>
-      <mass value="0.5"/>
-      <origin xyz="0 0 0.3"/>
-      <inertia ixx="0.02" iyy="0.02" izz="0.005" ixy="0" ixz="0" iyz="0"/>
+      <mass value="0.15"/>
+      <origin xyz="0 0 0"/>
+      <inertia ixx="2e-4" iyy="2e-4" izz="2e-4" ixy="0" ixz="0" iyz="0"/>
     </inertial>
     <visual>
-      <origin xyz="0 0 0.3"/>
-      <geometry><box size="0.08 0.2 0.6"/></geometry>
-      <material name="orange"><color rgba="1.0 0.5 0.0 1"/></material>
+      <geometry><box size="0.07 0.09 0.07"/></geometry>
+      <material name="gizmo_head"/>
     </visual>
     <collision>
-      <origin xyz="0 0 0.3"/>
-      <geometry><box size="0.08 0.2 0.6"/></geometry>
+      <geometry><box size="0.07 0.09 0.07"/></geometry>
     </collision>
   </link>
-  <joint name="paddle_joint" type="revolute">
-    <parent link="base_link"/>
-    <child link="paddle_link"/>
-    <origin xyz="0 0 0.1" rpy="0 0 0"/>
-    <axis xyz="0 1 0"/>
-    <limit lower="-1.57" upper="1.57" effort="20.0" velocity="2.0"/>
+  <joint name="head_fixed" type="fixed">
+    <parent link="body_link"/>
+    <child link="head_link"/>
+    <origin xyz="${body_x/2 - 0.02} 0 ${body_z/2 + 0.035}" rpy="0 0 0"/>
   </joint>
-  <!-- ros2_control hookup for Gazebo Harmonic via gz_ros2_control -->
-  <ros2_control name="GizmoSystem" type="system">
-    <hardware>
-      <plugin>gz_ros2_control/GazeboSimSystem</plugin>
-    </hardware>
-    <joint name="paddle_joint">
+  <!-- Four legs. -->
+  <xacro:gizmo_leg prefix="front_left"  parent="body_link"
+                   x="${ hip_x}" y="${ hip_y}" z="${hip_z}"/>
+  <xacro:gizmo_leg prefix="front_right" parent="body_link"
+                   x="${ hip_x}" y="${-hip_y}" z="${hip_z}"/>
+  <xacro:gizmo_leg prefix="rear_left"   parent="body_link"
+                   x="${-hip_x}" y="${ hip_y}" z="${hip_z}"/>
+  <xacro:gizmo_leg prefix="rear_right"  parent="body_link"
+                   x="${-hip_x}" y="${-hip_y}" z="${hip_z}"/>
+  <!-- Arms: one revolute joint each, swings forward/back around Y. -->
+  <xacro:macro name="gizmo_arm" params="prefix y_sign">
+    <link name="${prefix}_arm_link">
+      <inertial>
+        <mass value="0.08"/>
+        <origin xyz="0 0 -0.04"/>
+        <inertia ixx="2e-4" iyy="2e-4" izz="3e-5" ixy="0" ixz="0" iyz="0"/>
+      </inertial>
+      <visual>
+        <origin xyz="0 0 -0.04"/>
+        <geometry><box size="0.025 0.025 0.08"/></geometry>
+        <material name="gizmo_arm"/>
+      </visual>
+      <collision>
+        <origin xyz="0 0 -0.04"/>
+        <geometry><box size="0.025 0.025 0.08"/></geometry>
+      </collision>
+    </link>
+    <joint name="${prefix}_arm_joint" type="revolute">
+      <parent link="body_link"/>
+      <child link="${prefix}_arm_link"/>
+      <origin xyz="0 ${y_sign * (body_y/2 + 0.012)} ${body_z/2 - 0.015}" rpy="0 0 0"/>
+      <axis xyz="0 1 0"/>
+      <limit lower="-2.5" upper="2.5" effort="3.0" velocity="3.0"/>
+      <dynamics damping="0.05" friction="0.01"/>
+    </joint>
+  </xacro:macro>
+  <xacro:gizmo_arm prefix="left"  y_sign="1"/>
+  <xacro:gizmo_arm prefix="right" y_sign="-1"/>
+  <!-- ros2_control hookup for Gazebo Harmonic via gz_ros2_control. -->
+  <xacro:macro name="position_joint" params="name lower upper">
+    <joint name="${name}">
       <command_interface name="position">
-        <param name="min">-1.57</param>
-        <param name="max">1.57</param>
+        <param name="min">${lower}</param>
+        <param name="max">${upper}</param>
       </command_interface>
       <state_interface name="position"/>
@@ -57,4 +114,19 @@
       <state_interface name="effort"/>
     </joint>
+  </xacro:macro>
+  <ros2_control name="GizmoSystem" type="system">
+    <hardware>
+      <plugin>gz_ros2_control/GazeboSimSystem</plugin>
+    </hardware>
+    <xacro:position_joint name="front_left_hip_joint"   lower="-1.2" upper="1.2"/>
+    <xacro:position_joint name="front_left_knee_joint"  lower="-2.2" upper="0.2"/>
+    <xacro:position_joint name="front_right_hip_joint"  lower="-1.2" upper="1.2"/>
+    <xacro:position_joint name="front_right_knee_joint" lower="-2.2" upper="0.2"/>
+    <xacro:position_joint name="rear_left_hip_joint"    lower="-1.2" upper="1.2"/>
+    <xacro:position_joint name="rear_left_knee_joint"   lower="-2.2" upper="0.2"/>
+    <xacro:position_joint name="rear_right_hip_joint"   lower="-1.2" upper="1.2"/>
+    <xacro:position_joint name="rear_right_knee_joint"  lower="-2.2" upper="0.2"/>
+    <xacro:position_joint name="left_arm_joint"         lower="-2.5" upper="2.5"/>
+    <xacro:position_joint name="right_arm_joint"        lower="-2.5" upper="2.5"/>
   </ros2_control>
   <gazebo>

Commit message: Add arm actions, head pan and face panel (Iterations 3 & 4)
Iteration 3 (Arme & Winken polieren):
- Add wave_left, wave_right, arms_up, arms_down actions to
  gizmo_gait_node, all routed through the stand pose so the controller
  never sees a jump near the joint limits.
- New crawl_arm_action parameter overlays a wave or static arm pose
  on top of the crawl trajectory without disturbing the leg cycle.

Iteration 4 (Kopf, Display-Dummy, Gesichtsausdrücke):
- Replace the fixed head joint with a head_pan_joint (revolute around
  Z, +/-1.5 rad) and add a display_link panel on the head's front face.
- Attach a gz-sim-material-color-system plugin to display_link so the
  visual is retinted whenever a gz.msgs.Color arrives on
  /gizmo/face_color. ros_gz_bridge bridges std_msgs/ColorRGBA to that
  topic.
- New gizmo_face_node maps /gizmo/face strings (neutral, happy, sad,
  surprised, angry) to ColorRGBA values and latches the default
  expression at startup.
- ros2_control block, JTC config and JOINT_ORDER updated for the new
  head_pan_joint.

File: src/gizmo_description/urdf/gizmo.urdf.xacro (robot description, xacro)
@@ -2,5 +2,6 @@
 <robot name="gizmo" xmlns:xacro="http://www.ros.org/wiki/xacro">
   <!--
-    Iteration 1 Gizmo: a simple quadruped with two arms.
+    Gizmo: simple quadruped with two arms, a panning head and a
+    colour-controlled face panel.
     Joints exposed to ros2_control:
       front_left_hip_joint, front_left_knee_joint
@@ -9,4 +10,7 @@
       rear_right_hip_joint, rear_right_knee_joint
       left_arm_joint, right_arm_joint
+      head_pan_joint
+    The display_link visual on the head is retinted at runtime by the
+    Gazebo MaterialColor system listening on /gizmo/face_color.
     Geometry is deliberately box/cylinder/sphere only - this is here
     to validate URDF, controllers and gait scaffolding, not to look
@@ -45,5 +49,9 @@
     <origin xyz="0 0 0" rpy="0 0 0"/>
   </joint>
-  <!-- Head: fixed for now, gets a joint in a later iteration. -->
+  <!-- Head: pans around Z so Gizmo can look left/right.
+       Geometry stays a simple box; real CAD lands later. -->
+  <xacro:property name="head_x" value="0.07"/>
+  <xacro:property name="head_y" value="0.09"/>
+  <xacro:property name="head_z" value="0.07"/>
   <link name="head_link">
     <inertial>
@@ -53,16 +61,53 @@
     </inertial>
     <visual>
-      <geometry><box size="0.07 0.09 0.07"/></geometry>
+      <geometry><box size="${head_x} ${head_y} ${head_z}"/></geometry>
       <material name="gizmo_head"/>
     </visual>
     <collision>
-      <geometry><box size="0.07 0.09 0.07"/></geometry>
+      <geometry><box size="${head_x} ${head_y} ${head_z}"/></geometry>
     </collision>
   </link>
-  <joint name="head_fixed" type="fixed">
+  <joint name="head_pan_joint" type="revolute">
     <parent link="body_link"/>
     <child link="head_link"/>
     <origin xyz="${body_x/2 - 0.02} 0 ${body_z/2 + 0.035}" rpy="0 0 0"/>
+    <axis xyz="0 0 1"/>
+    <limit lower="-1.5" upper="1.5" effort="2.0" velocity="2.0"/>
+    <dynamics damping="0.05" friction="0.01"/>
   </joint>
+  <!-- Display panel sitting on the front face of the head. The visual
+       is named so the Gazebo MaterialColor system below can retint it
+       in response to /gizmo/face_color messages. No collision: this is
+       a cosmetic surface, and a thin collision causes contact noise. -->
+  <link name="display_link">
+    <inertial>
+      <mass value="0.01"/>
+      <origin xyz="0 0 0"/>
+      <inertia ixx="1e-6" iyy="1e-6" izz="1e-6" ixy="0" ixz="0" iyz="0"/>
+    </inertial>
+    <visual name="display_visual">
+      <geometry><box size="0.005 0.06 0.045"/></geometry>
+      <material name="gizmo_face"/>
+    </visual>
+  </link>
+  <joint name="display_fixed" type="fixed">
+    <parent link="head_link"/>
+    <child link="display_link"/>
+    <origin xyz="${head_x/2 + 0.0026} 0 0" rpy="0 0 0"/>
+  </joint>
+  <!-- Gazebo Harmonic MaterialColor system: retint display_link's
+       visual whenever a gz.msgs.Color message arrives on the topic.
+       The face node publishes std_msgs/ColorRGBA which is bridged to
+       gz.msgs.Color by ros_gz_bridge in the launch file. -->
+  <gazebo reference="display_link">
+    <plugin filename="gz-sim-material-color-system"
+            name="gz::sim::systems::MaterialColor">
+      <topic>/gizmo/face_color</topic>
+      <ambient>0.7 0.7 0.75 1</ambient>
+      <diffuse>0.7 0.7 0.75 1</diffuse>
+      <specular>0.2 0.2 0.2 1</specular>
+      <emissive>0.4 0.4 0.45 1</emissive>
+    </plugin>
+  </gazebo>
   <!-- Four legs. -->
   <xacro:gizmo_leg prefix="front_left"  parent="body_link"
@@ -129,4 +174,5 @@
     <xacro:position_joint name="left_arm_joint"         lower="-2.5" upper="2.5"/>
     <xacro:position_joint name="right_arm_joint"        lower="-2.5" upper="2.5"/>
+    <xacro:position_joint name="head_pan_joint"         lower="-1.5" upper="1.5"/>
   </ros2_control>
   <gazebo>

File: src/gizmo_description/urdf/materials.xacro (robot description, xacro)
@@ -16,3 +16,9 @@
     <color rgba="0.55 0.35 0.10 1.0"/>
   </material>
+  <!-- Initial colour of the face display. The MaterialColor Gazebo
+       system retints this material at runtime when /gizmo/face_color
+       is published, so the value here is just the boot-time look. -->
+  <material name="gizmo_face">
+    <color rgba="0.7 0.7 0.75 1.0"/>
+  </material>
 </robot>
